File: motherboard/pcb.kicad_sch (KiCad schematic)
At the start: 132 parts, among them CN1 Conn_01x12, CN2 Conn_01x10, IC11 MK4164N, IC12 MK4164N, IC13 MK4164N, IC14 MK4164N, IC18 74LS245, IC30 8255A, IC31 74LS245, IC41 74LS245, IC42 74LS273, IC43 74LS174, IC6 MK4164N, IC7 MK4164N, IC8 MK4164N, IC9 MK4164N, SW1 SW_DIP_x08, U1 Z84C00xxP, U2 MK4116N, X1 32.768, X2 15974.4, X3 1431818, ic10 74LS157, ic15 74LS273, ic16 74LS273, ic17 74LS367, ic19 74LS138, ic20 74LS245, ic21 74LS245, ic22 D8257, ic23 B6102C005, ic24 D1990AC, ic25 LS32, ic26 LS32, ic27 LS32, ic28 74LS373, ic29 74LS373, ic32 B6102C006, ic33 74LS245, ic34 74LS245, ic37 74LS08, ic38 74LS14, ic39 74LS00, ic4 74LS10, ic40 7407, ic44 74LS32, ic45 74LS00, ic46 B6102C007, ic47 B6102C008, ic48 74LS393, ic49 74LS153, ic5 74LS157, ic50 74LS153, ic51 LS04, ic52 74LS00, ic53 MC1489PG, ic54 D8251, ic58 D3301AC, ic60 MK4116N, ic61 MC1488N, ic64 MK4116N, ic65 MK4116N, ic66 4013, ic67 4081, ic68 4030, ic71 MK4116N, ic72 MK4116N, ic75 74LS86, ic76 74LS145, ic77 MK4116N, ic78 MK4116N, ic79 7406, ic80 7428, ic81 74LS245, ic82 74LS245

Commit message: Add files via upload
Parts:
- added ic3: 2764, Package_DIP:DIP-28_W15.24mm, symbol Memory_EPROM:2764
- added ic56: 74LS153, symbol 74xx:74LS153
- added ic57: D2316, Package_DIP:DIP-24_W15.24mm, symbol New_Library:D2316
- added ic62, ic63: 74LS157, symbol 74xx:74LS157
- added ic70: 74LS175, symbol 74xx:74LS175
- renumbered rom1 to ic1, rom2 to ic2
Connections:
- net GND: now also ic56.1 (Ea), ic56.15 (Eb), ic57.18 (~{CE2}), ic57.20 (~{CE1}), ic62.15 (E), ic63.15 (E); no longer ic47.21 (Pin_21)
- net VCC: now also ic57.21 (~{CE3})
- net ic46_23: now reaches ic46.23 (Pin_23)
- net ic46_23: now also ic62.1 (S), ic63.1 (S)
- net ic46_29: now reaches ic46.29 (Pin_29)
- net ic46_29: now also ic70.9 (Cp)
- net ic46_3: now reaches ic46.3 (Pin_3)
- net ic46_3: now also ic70.4 (D0)
- net ic46_4: now reaches ic46.4 (Pin_4)
- net ic46_4: now also ic70.5 (D1)
- net ic46_5: now reaches ic46.5 (Pin_5)
- net ic46_5: now also ic70.12 (D2)
- net ic46_6: now reaches ic46.6 (Pin_6)
- net ic46_6: now also ic70.13 (D3)
- net rom3_oe: now reaches ic4.13, ic4.2, ic4.6
- net rom3_oe: now also ic3.22 (~{OE})
- new net: ic57.11 (D2), ic62.11 (I0c)
- new net: ic57.13 (D3), ic62.14 (I0d)
- new net: ic57.9 (D0), ic62.2 (I0a)
- new net: ic57.10 (D1), ic62.5 (I0b)
- new net: ic57.14 (D4), ic63.2 (I0a)
- new net: ic57.15 (D5), ic63.5 (I0b)
- new net: ic57.16 (D6), ic63.11 (I0c)
- new net: ic57.17 (D7), ic63.14 (I0d)
- new net chr_a0: ic57.8 (A0), ic70.2 (Q0)
- new net chr_a1: ic57.7 (A1), ic70.7 (Q1)
- new net chr_a10: ic56.13 (I3b), ic57.19 (A10)
- new net chr_a2: ic57.6 (A2), ic70.10 (Q2)
- new net chr_a3: ic56.6 (I0a), ic57.5 (A3)
- new net chr_a4: ic56.5 (I1a), ic57.4 (A4)
- new net chr_a5: ic56.4 (I2a), ic57.3 (A5)
- new net chr_a6: ic56.3 (I3a), ic57.2 (A6)
- new net chr_a7: ic56.10 (I0b), ic57.1 (A7)
- new net chr_a8: ic56.11 (I1b), ic57.23 (A8)
- new net chr_a9: ic56.12 (I2b), ic57.22 (A9)
- new net ic47_21: ic47.21 (Pin_21), ic70.1 (~{Mr})
Other:
- note added: "CHR_ROM"
- note added: "ROM1"
- note added: "ROM2"
- note added: "ROM3"
- moved on the sheet: IC18

Commit message: Add files via upload
Parts:
- added R21: 1K, symbol Device:R_Small
- added READER: DE9_Pins, symbol Connector:DE9_Pins
- added unit 2 of ic37
Connections:
- net GND: now also READER.5, READER.7
- net VCC: now also R21.1, READER.9
- net bus_int2: now also ic37.5
- net prnt_9: now also READER.6
- net ic23_17: now reaches ic23.17 (Pin_17)
- net ic23_17: now also ic37.6
- net DB9_3: now reaches ic16.16 (Q6)
- net DB9_3: now also READER.3
- net DB9_4: now reaches ic16.19 (Q7)
- net DB9_4: now also READER.4
- net at IC41.12 (B6), MR5.8 (R7): now also READER.2
- net at IC41.11 (B7), MR5.9 (R8): now also READER.1
- new net: R21.2, READER.8, ic37.4
Other:
- moved on the sheet: R22, ic32

Commit message: Add files via upload
Parts:
- removed unit 4 of ic4
- added ic36, ic73: LM311, symbol Comparator:LM311
- added unit 4 of ic37
- added unit 1 of ic38
- added unit 5 of ic38
- added unit 4 of ic38
- added unit 6 of ic38
- added unit 2 of ic38
- added unit 3 of ic39
- added unit 4 of ic39
- added unit 5 of ic40
- added unit 4 of ic40
- added unit 3 of ic40
- added unit 1 of ic44
- added unit 2 of ic44
- added unit 4 of ic44
- added unit 2 of ic51
- added unit 1 of ic51
- added unit 4 of ic52
- added ic55: 74LS166, symbol 74xx:74LS166
- added unit 2 of ic66
- added unit 2 of ic67
- added unit 1 of ic67
- added unit 3 of ic68
- added ic69: 4024, symbol 4xxx_IEEE:4024
- added ic74: 4013, symbol 4xxx:4013
- added unit 3 of ic75
- added unit 2 of ic75
- added unit 4 of ic75
- added unit 5 of ic79
- added unit 4 of ic79
Connections:
- net ic46_33: now also ic40.10
- net ic47_21: now also ic39.5
- net ic47_25: now also ic51.3
- net reset1: now also ic38.3
- net reset2: now also ic38.4
- net /dack0: now also ic39.12
- net /dack1: now also ic39.13
- net at ic23.24 (Pin_24): now also ic38.2
- net ic23_39: now reaches ic23.39 (Pin_39)
- net ic23_39: now also ic25.10
- net at ic25.9, ic37.1: now also ic27.1, ic38.8
- net ic32_6: now reaches ic27.2, ic37.2
- net ic32_6: now also ic32.6 (Pin_6)
- net /bus_memr: now reaches CPU_BUS.b21 (Pin_b21), ic39.4
- net at ic39.6: now also ic44.13, ic44.2
- net /bus_ras0: now reaches CPU_BUS.a26 (Pin_a26)
- net /bus_ras0: now also ic44.11
- net /bus_ras1: now reaches CPU_BUS.a27 (Pin_a27)
- net /bus_ras1: now also ic44.3
- net /DMATC: now reaches CPU_BUS.b26 (Pin_b26)
- net /DMATC: now also ic39.8
- net ic32_34: now reaches ic32.34 (Pin_34)
- net ic32_34: now also ic44.12
- net ic32_35: now reaches ic32.35 (Pin_35)
- net ic32_35: now also ic44.1
- net hrq: now reaches ic22.10 (Pin_10)
- net hrq: now also ic37.13, ic51.1
- net DRQ1: now reaches ic22.18 (Pin_18)
- net DRQ1: now also ic38.12
- net TC: now reaches ic22.36 (Pin_36)
- net TC: now also ic39.9
- net HLDA: now reaches ic22.7 (Pin_7)
- net HLDA: now also ic37.11
- new net: ic37.12, ic51.4
- new net: ic40.11, ic51.2
- new net: ic40.6, ic40.8
- new net: ic39.10, ic39.11
- no-connect marks 9 -> 12
Other:
- moved on the sheet: R22, ic25C, ic27A, ic32, ic39B, ic44C

Commit message: Add files via upload
Parts:
- removed ic22: D8257, symbol Connector_Generic:Conn_02x20_Counter_Clockwise
- removed ic54: D8251, symbol Connector_Generic:Conn_02x14_Counter_Clockwise
- removed ic58: D3301AC, symbol Connector_Generic:Conn_02x20_Counter_Clockwise
- added C79: 220p, symbol Device:C_Small
- added C80, C81: 470p, symbol Device:C_Small
- added D5: D, symbol Device:D
- added IC54: 8251, Package_DIP:DIP-28_W15.24mm, symbol New_Library:8251
- added IC58: D3301AC, Package_DIP:DIP-40_W15.24mm, symbol New_Library:uPD3301
- added R25, R59, R63, R65: ~, symbol Device:R_Small
- added R45: 2.2k, symbol Device:R_Small
- added R47: (no value), symbol Device:R_Small
- added R48: 15k, symbol Device:R_Small
- added RESET: ~, Button_Switch_SMD:Nidec_Copal_CAS-120A, symbol Switch:SW_Nidec_CAS-120A1
- added ic22: D8257, Package_DIP:DIP-40_W15.24mm, symbol New_Library:C8257_D8257_P8257_AM8557
- JSW: value Conn_02x08_Top_Bottom -> RS-232C
- SW1: value SW_DIP_x08 -> MODE SELECT
- renumbered U1 to ic35
Connections:
- net V1 is gone; now on net /DRQ1: CPU_BUS.a35 (Pin_a35)
- net 8255_rd: now also IC54.13 (~{RD}), IC58.9 (RD)
- net 8255_wr: now also IC54.10 (~{WR})
- net 8257_clk: now also ic22.12 (CLK)
- net 8257_cs: now also ic22.11 (/CS)
- net D3301_cs: now also IC58.11 (/CS)
- net DRQ1: now also ic22.18 (DRQ1)
- net GND: now also ic55.1 (Ds), ic55.6 (CE), ic66.10 (R), ic66.11 (C), ic66.8 (S), ic66.9 (D), ic68.6, C79.2, C80.2, C81.2, RESET.1 (C), ic22.16 (DRQ3)
- net HLDA: now also ic22.7 (HLDA)
- net TC: now also ic22.36 (TC)
- net VCC: now also D5.1 (K), R25.2, R59.2
- net a0: now also ic22.32 (A0)
- net a1: now also ic22.33 (A1)
- net a2: now also ic22.34 (A2)
- net a3: now also ic22.35 (A3)
- net a4: now also ic22.37 (A4)
- net a5: now also ic22.38 (A5)
- net a6: now also ic22.39 (A6)
- net a7: now also ic22.40 (A7)
- net bsclock: now also ic69.1 (~{CLK})
- net d0: now also IC54.27 (D0), IC58.12 (DB0), ic22.30 (D0)
- net d1: now also IC54.28 (D1), IC58.13 (DB1), ic22.29 (D1)
- net d2: now also IC54.1 (D2), IC58.14 (DB2), ic22.28 (D2)
- net d3: now also IC54.2 (D3), IC58.15 (DB3), ic22.27 (D3)
- net d4: now also IC54.5 (D4), IC58.16 (DB4), ic22.26 (D4)
- net d5: now also IC54.6 (D5), IC58.17 (DB5), ic22.23 (D5)
- net d6: now also IC54.7 (D6), IC58.18 (DB6), ic22.22 (D6)
- net d7: now also IC54.8 (D7), IC58.19 (DB7), ic22.21 (D7)
- net hrq: now also ic22.10 (HRQ)
- net ic23_1: now also IC54.12 (C/~{D})
- net memwr1: now also ic22.4 (/MEMW)
- net reset2: now also ic22.13 (RESET)
- net /bus_memr: now also ic34.2 (A0)
- net /dack0: now also ic22.25 (/DACK0)
- net /dack1: now also ic22.24 (/DACK1)
- net at ic38.1: now also D5.2 (A), R25.1, RESET.2 (B)
- net at ic74.2 (~{Q}): now also ic68.5
- net at ic74.3 (C): now also ic74.10 (R)
- net at ic74.4 (R): now also ic74.6 (S), ic74.8 (S), ic74.9 (D)
- net at ic74.5 (D): now also ic74.13 (Q)
- net at ic67.4: now also ic68.8
- net at ic67.5: now also ic67.6, R48.2
- net ic46_24: now reaches ic46.24 (Pin_24)
- net ic46_24: now also ic55.15 (PE)
- net ic46_26: now reaches ic46.26 (Pin_26)
- net ic46_26: now also ic55.13 (Qh)
- net ic46_27: now reaches ic46.27 (Pin_27)
- net ic46_27: now also ic55.7 (Clk)
- net at ic68.10: now also ic69.2 (MR)
- net at ic68.9: now also R47.1
- net at IC43.15 (Q5), ic45.13, ic49.2 (S1)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: now also ic40.9
- net at ic28.1 (OE), ic38.6, ic39.1: now also ic38.9
- net AEN: now reaches ic29.1 (OE), ic38.5
- net AEN: now also ic22.9 (AEN)
- net at ic74.11 (C): now also ic67.3
- net DRQ0: now reaches ic38.10
- net DRQ0: now also ic22.19 (DRQ0)
- net /DRQ0: now reaches ic38.11
- net /DRQ0: now also CPU_BUS.b28 (Pin_b28)
- net at ic69.5 (Q4): now also ic67.1
- net at ic69.6 (Q3): now also ic67.2, ic68.1
- net at ic69.9 (Q2): now also ic68.12
- net at ic68.2: now also C81.1
- net at ic79.10: now also R63.2
- net at ic79.11: now also ic80.6
- net TxD: now reaches ic51.9, ic67.8
- net TxD: now also IC54.19 (TxD)
- net at ic79.8: now also R65.1
- net at ic79.9: now also ic80.8
- net at ic73.2 (+): now also R45.1
- net at ic68.13: now also C80.1
- net at ic62.12 (Zd): now also ic55.5 (D)
- net at ic62.13 (I1d): now also ic56.9 (Zb), ic62.3 (I1a), ic62.6 (I1b)
- net at ic62.4 (Za): now also ic55.2 (A)
- net at ic62.7 (Zb): now also ic55.3 (B)
- net at ic62.9 (Zc): now also ic55.4 (C)
- net DSR: now reaches ic53.11 (OUT_D)
- net DSR: now also IC54.22 (~{DSR})
- net at ic53.6 (OUT_B): now also ic40.5
- net ic32_27: now reaches ic32.27 (Pin_27)
- net ic32_27: now also IC54.20 (CLK)
- net RxC: now reaches ic49.9 (Zb)
- net RxC: now also IC54.25 (~{RxC})
- net RxD: now reaches ic50.7 (Za)
- net RxD: now also IC54.3 (RxD)
- net TxC: now reaches ic49.7 (Za)
- net TxC: now also IC54.9 (~{TxC})
- net at ic63.12 (Zd): now also ic55.14 (H)
- net at ic63.13 (I1d): now also ic56.7 (Za), ic63.3 (I1a), ic63.6 (I1b)
- net at ic63.4 (Za): now also ic55.10 (E)
- net at ic63.7 (Zb): now also ic55.11 (F)
- net at ic63.9 (Zc): now also ic55.12 (G)
- net /DRQ1: now reaches ic38.13
- net at ic70.14 (~{Q3}): now also ic55.9 (Clr)
- net 8251_11 renamed 8251_cs
- net 8251_cs: now also IC54.11 (~{CS})
- net V2 renamed /bus_dack1
- net ic32_3 renamed IOR
- net IOR: now also ic22.1 (/IOR)
- new net: R59.1, R65.2
- new net: C79.1, R47.2
- new net: R45.2, R48.1
- new net DRQ2: IC58.6 (DRQ), ic22.17 (DRQ2)
- new net IOW: IC58.10 (WR), ic22.2 (/IOW)
- new net /dack2: IC58.7 (DACK), ic22.14 (/DACK2)
- no-connect marks 12 -> 37
Other:
- note added: "1 2 3 4 5 6 7 8"
- note added: "8 7 6 5 4 3 2 1"
- moved on the sheet: C35, C36, C37, C40, C43, C44, C45, C46, CPU_BUS, IC42, R23, R24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
